File: power.kicad_sch (KiCad schematic)
At the start: 26 parts, among them J201 Power_Planes, Q201 Q_PMOS_GSD, U201 AP2112K-3.3, U203 AMS1117-3.3

Commit message: Updated PCB after DRC. Updated Connector lib.
Parts:
- added R211: 0, Resistor_SMD:R_1206_3216Metric_Pad1.30x1.75mm_HandSolder, symbol Device:R
Connections:
- net GND: now also R211.1
- net GNDA: now also R211.2
Changed lines of the file:
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@@
   (junction (at 123.19 49.53) (diameter 0) (color 0 0 0 0)
   )
+  (junction (at 227.33 48.26) (diameter 0) (color 0 0 0 0)
+  )
   (junction (at 191.77 91.44) (diameter 0) (color 0 0 0 0)
   )
@@
   (junction (at 69.85 50.8) (diameter 0) (color 0 0 0 0)
   )
+  (junction (at 264.16 48.26) (diameter 0) (color 0 0 0 0)
+  )
   (junction (at 264.16 35.56) (diameter 0) (color 0 0 0 0)
   )
@@
     (stroke (width 0) (type default) (color 0 0 0 0))
   )
+  (wire (pts (xy 248.92 48.26) (xy 264.16 48.26))
+    (stroke (width 0) (type default) (color 0 0 0 0))
+  )
   (wire (pts (xy 76.2 114.3) (xy 95.25 114.3))
     (stroke (width 0) (type default) (color 0 0 0 0))
@@
     (stroke (width 0) (type default) (color 0 0 0 0))
   )
+  (wire (pts (xy 227.33 48.26) (xy 241.3 48.26))
+    (stroke (width 0) (type default) (color 0 0 0 0))
+  )
   (wire (pts (xy 83.82 100.33) (xy 95.25 100.33))
     (stroke (width 0) (type default) (color 0 0 0 0))
@@
     (stroke (width 0) (type default) (color 0 0 0 0))
   )
+  (wire (pts (xy 227.33 48.26) (xy 227.33 52.07))
+    (stroke (width 0) (type default) (color 0 0 0 0))
+  )
   (wire (pts (xy 95.25 24.13) (xy 95.25 30.48))
     (stroke (width 0) (type default) (color 0 0 0 0))
@@
     (stroke (width 0) (type default) (color 0 0 0 0))
   )
-  (wire (pts (xy 264.16 45.72) (xy 264.16 52.07))
+  (wire (pts (xy 264.16 45.72) (xy 264.16 48.26))
     (stroke (width 0) (type default) (color 0 0 0 0))
   )
@@
     (stroke (width 0) (type default) (color 0 0 0 0))
   )
-  (wire (pts (xy 227.33 45.72) (xy 227.33 52.07))
+  (wire (pts (xy 227.33 45.72) (xy 227.33 48.26))
     (stroke (width 0) (type default) (color 0 0 0 0))
   )
@@
   )
   (wire (pts (xy 187.96 91.44) (xy 191.77 91.44))
+    (stroke (width 0) (type default) (color 0 0 0 0))
+  )
+  (wire (pts (xy 264.16 48.26) (xy 264.16 52.07))
     (stroke (width 0) (type default) (color 0 0 0 0))
   )
@@
       (effects (font (size 1.27 1.27)) hide)
     )
+    (pin "1")
+    (pin "2")
+  )
+  (symbol (lib_id "Device:R") (at 245.11 48.26 90) (unit 1)
+    (in_bom yes) (on_board yes)
+    (property "Reference" "R211" (id 0) (at 243.9416 46.482 0)
+      (effects (font (size 1.27 1.27)) (justify left))
+    )
+    (property "Value" "0" (id 1) (at 246.253 46.482 0)
+      (effects (font (size 1.27 1.27)) (justify left))
+    )
+    (property "Footprint" "Resistor_SMD:R_1206_3216Metric_Pad1.30x1.75mm_HandSolder" (id 2) (at 245.11 50.038 90)
+      (effects (font (size 1.27 1.27)) hide)
+    )
+    (property "Datasheet" "~" (id 3) (at 245.11 48.26 0)
+      (effects (font (size 1.27 1.27)) hide)
+    )

Commit message: Updated all but polyfuse and ferride bead to correct footprints.
Parts:
- added R204: 100R, Resistor_SMD:R_0603_1608Metric_Pad0.98x0.95mm_HandSolder, symbol Device:R
- D201: value D_Zener -> BZX284-C5V1; footprint Diode_SMD:D_0805_2012Metric_Pad1.15x1.40mm_HandSolder -> Diode_SMD:D_SOD-110
- Q201: value Q_PMOS_GSD -> SI4435DY_GSD; footprint Package_TO_SOT_SMD:TSOT-23 -> Package_SO:SOIC-8_3.9x4.9mm_P1.27mm
Connections:
- net GND: now also R204.2; no longer D201.2 (A), Q201.1 (G)
- new net: D201.2 (A), Q201.1 (G), R204.1
Changed lines of the file:
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@@
   (junction (at 49.53 148.59) (diameter 0) (color 0 0 0 0)
   )
-  (junction (at 82.55 40.64) (diameter 0) (color 0 0 0 0)
-  )
   (junction (at 52.07 100.33) (diameter 0) (color 0 0 0 0)
   )
+  (junction (at 90.17 40.64) (diameter 0) (color 0 0 0 0)
+  )
   (junction (at 214.63 104.14) (diameter 0) (color 0 0 0 0)
   )
@@
     (stroke (width 0) (type default) (color 0 0 0 0))
   )
+  (wire (pts (xy 90.17 40.64) (xy 90.17 43.18))
+    (stroke (width 0) (type default) (color 0 0 0 0))
+  )
   (wire (pts (xy 180.34 93.98) (xy 180.34 91.44))
     (stroke (width 0) (type default) (color 0 0 0 0))
@@
     (stroke (width 0) (type default) (color 0 0 0 0))
   )
-  (wire (pts (xy 69.85 50.8) (xy 82.55 50.8))
+  (wire (pts (xy 69.85 50.8) (xy 90.17 50.8))
     (stroke (width 0) (type default) (color 0 0 0 0))
   )
@@
     (stroke (width 0) (type default) (color 0 0 0 0))
   )
-  (wire (pts (xy 95.25 40.64) (xy 82.55 40.64))
+  (wire (pts (xy 95.25 40.64) (xy 90.17 40.64))
     (stroke (width 0) (type default) (color 0 0 0 0))
   )
@@
     (stroke (width 0) (type default) (color 0 0 0 0))
   )
-  (wire (pts (xy 82.55 40.64) (xy 82.55 50.8))
-    (stroke (width 0) (type default) (color 0 0 0 0))
-  )
   (wire (pts (xy 180.34 91.44) (xy 187.96 91.44))
     (stroke (width 0) (type default) (color 0 0 0 0))
@@
   )
   (wire (pts (xy 76.2 107.95) (xy 76.2 114.3))
+    (stroke (width 0) (type default) (color 0 0 0 0))
+  )
+  (wire (pts (xy 90.17 40.64) (xy 82.55 40.64))
     (stroke (width 0) (type default) (color 0 0 0 0))
   )
@@
     (in_bom yes) (on_board yes)
     (property "Reference" "Q201" (id 0) (at 82.55 24.3332 90))
-    (property "Value" "Q_PMOS_GSD" (id 1) (at 82.55 26.6446 90))
-    (property "Footprint" "Package_TO_SOT_SMD:TSOT-23" (id 2) (at 80.01 27.94 0)
+    (property "Value" "SI4435DY_GSD" (id 1) (at 82.55 26.6446 90))
+    (property "Footprint" "Package_SO:SOIC-8_3.9x4.9mm_P1.27mm" (id 2) (at 80.01 27.94 0)
       (effects (font (size 1.27 1.27)) hide)
     )
@@
       (effects (font (size 1.27 1.27)) (justify left))
     )
-    (property "Value" "D_Zener" (id 1) (at 97.282 36.703 90)
-      (effects (font (size 1.27 1.27)) (justify left))
-    )
-    (property "Footprint" "Diode_SMD:D_0805_2012Metric_Pad1.15x1.40mm_HandSolder" (id 2) (at 95.25 35.56 0)
+    (property "Value" "BZX284-C5V1" (id 1) (at 97.282 36.703 90)
+      (effects (font (size 1.27 1.27)) (justify left))
+    )
+    (property "Footprint" "Diode_SMD:D_SOD-110" (id 2) (at 95.25 35.56 0)
       (effects (font (size 1.27 1.27)) hide)
     )
@@
     (pin "1")
   )
+  (symbol (lib_id "Device:R") (at 90.17 46.99 0) (unit 1)
+    (in_bom yes) (on_board yes)
+    (property "Reference" "R204" (id 0) (at 91.948 45.8216 0)
+      (effects (font (size 1.27 1.27)) (justify left))
+    )
+    (property "Value" "100R" (id 1) (at 91.948 48.133 0)
+      (effects (font (size 1.27 1.27)) (justify left))
+    )
+    (property "Footprint" "Resistor_SMD:R_0603_1608Metric_Pad0.98x0.95mm_HandSolder" (id 2) (at 88.392 46.99 90)
+      (effects (font (size 1.27 1.27)) hide)
+    )
+    (property "Datasheet" "~" (id 3) (at 90.17 46.99 0)
+      (effects (font (size 1.27 1.27)) hide)
+    )
+    (pin "1")
+    (pin "2")
+  )
   (symbol (lib_id "power:GND") (at 76.2 118.11 0) (unit 1)
