File: ovvekit.kicad_sch (KiCad schematic)
At the start: 32 parts, among them J1 ESP_PROG_JTAG, J2 ESP_PROG_UART, SW1 SW_Push, SW2 SW_Push, SW3 SW_Push, SW4 SW_Push, U1 ESP32-WROOM-32

Commit message: Updated PCB after DRC. Updated Connector lib.
Connections:
- net EN is gone; now on net RESET: J2.1 (EN)
Changed lines of the file:
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@@
     )
   )
-  (global_label "EN" (shape input) (at 224.79 144.78 180) (fields_autoplaced)
+  (global_label "RESET" (shape input) (at 224.79 144.78 180) (fields_autoplaced)
     (effects (font (size 1.27 1.27)) (justify right))
-    (property "Intersheet References" "${INTERSHEET_REFS}" (id 0) (at 0 0 0)
-      (effects (font (size 1.27 1.27)) hide)
+    (property "Intersheet References" "${INTERSHEET_REFS}" (id 0) (at 216.7206 144.7006 0)
+      (effects (font (size 1.27 1.27)) (justify right) hide)
     )
   )
@@
       (reference "#PWR0123") (unit 1) (value "GNDA") (footprint "")
     )
-    (path "/00000000-0000-0000-0000-00006099554c/00000000-0000-0000-0000-000061b361f4"
-      (reference "#PWR0124") (unit 1) (value "GND") (footprint "")
-    )
-    (path "/00000000-0000-0000-0000-00006099554c/00000000-0000-0000-0000-000061b386c1"
-      (reference "#PWR0125") (unit 1) (value "+3.3V") (footprint "")
-    )
-    (path "/00000000-0000-0000-0000-00006099554c/00000000-0000-0000-0000-000061b3eef1"
-      (reference "#PWR0126") (unit 1) (value "GND") (footprint "")
-    )
-    (path "/00000000-0000-0000-0000-00006099554c/00000000-0000-0000-0000-000061b400c0"
-      (reference "#PWR0127") (unit 1) (value "GND") (footprint "")
-    )
-    (path "/00000000-0000-0000-0000-00006099554c/00000000-0000-0000-0000-000061b458d5"
-      (reference "#PWR0128") (unit 1) (value "GND") (footprint "")
-    )
     (path "/00000000-0000-0000-0000-0000609974e9/00000000-0000-0000-0000-0000615dbfa4"
       (reference "#PWR0201") (unit 1) (value "+3.3V") (footprint "")
@@
       (reference "R210") (unit 1) (value "10") (footprint "Resistor_SMD:R_1206_3216Metric_Pad1.30x1.75mm_HandSolder")
     )
+    (path "/00000000-0000-0000-0000-0000609974e9/e5f46ad9-2ec1-46e2-9d32-c83596a7eaeb"
+      (reference "R211") (unit 1) (value "0") (footprint "Resistor_SMD:R_1206_3216Metric_Pad1.30x1.75mm_HandSolder")
+    )
     (path "/00000000-0000-0000-0000-0000609974e9/00000000-0000-0000-0000-000061afc736"
       (reference "R220") (unit 1) (value "100K") (footprint "Resistor_SMD:R_0603_1608Metric_Pad0.98x0.95mm_HandSolder")
@@
       (reference "U201") (unit 1) (value "AP2112K-3.3") (footprint "Package_TO_SOT_SMD:SOT-23-5")
     )
-    (path "/00000000-0000-0000-0000-00006099554c/00000000-0000-0000-0000-000061b29b38"
-      (reference "U202") (unit 1) (value "LSM6DS3") (footprint "Package_LGA:LGA-14_3x2.5mm_P0.5mm_LayoutBorder3x4y")
-    )
     (path "/00000000-0000-0000-0000-0000609974e9/6f094073-8ef6-4c6e-b324-ff1cd5f09bba"

Commit message: Updated all but polyfuse and ferride bead to correct footprints.
Parts:
- SW1, SW2, SW3: footprint Button_Switch_SMD:SW_Push_1P1T_NO_6x6mm_H9.5mm -> Button_Switch_THT:SW_PUSH_6mm_H5mm
- SW4: footprint Button_Switch_SMD:SW_Push_1P1T_NO_6x6mm_H9.5mm -> Button_Switch_SMD:SW_SPST_TL3342
Changed lines of the file:
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@@
     (property "Reference" "SW1" (id 0) (at 191.77 22.3225 0))
     (property "Value" "SW_Push" (id 1) (at 191.77 25.0976 0))
-    (property "Footprint" "Button_Switch_SMD:SW_Push_1P1T_NO_6x6mm_H9.5mm" (id 2) (at 191.77 24.13 0)
+    (property "Footprint" "Button_Switch_THT:SW_PUSH_6mm_H5mm" (id 2) (at 191.77 24.13 0)
       (effects (font (size 1.27 1.27)) hide)
     )
@@
     (property "Reference" "SW2" (id 0) (at 191.77 42.6425 0))
     (property "Value" "SW_Push" (id 1) (at 191.77 45.4176 0))
-    (property "Footprint" "Button_Switch_SMD:SW_Push_1P1T_NO_6x6mm_H9.5mm" (id 2) (at 191.77 44.45 0)
+    (property "Footprint" "Button_Switch_THT:SW_PUSH_6mm_H5mm" (id 2) (at 191.77 44.45 0)
       (effects (font (size 1.27 1.27)) hide)
     )
@@
     (property "Reference" "SW3" (id 0) (at 246.38 25.781 0))
     (property "Value" "SW_Push" (id 1) (at 246.38 28.0924 0))
-    (property "Footprint" "Button_Switch_SMD:SW_Push_1P1T_NO_6x6mm_H9.5mm" (id 2) (at 246.38 27.94 0)
+    (property "Footprint" "Button_Switch_THT:SW_PUSH_6mm_H5mm" (id 2) (at 246.38 27.94 0)
       (effects (font (size 1.27 1.27)) hide)
     )
@@
     (property "Reference" "SW4" (id 0) (at 247.65 58.801 0))
     (property "Value" "SW_Push" (id 1) (at 247.65 61.1124 0))
-    (property "Footprint" "Button_Switch_SMD:SW_Push_1P1T_NO_6x6mm_H9.5mm" (id 2) (at 247.65 60.96 0)
+    (property "Footprint" "Button_Switch_SMD:SW_SPST_TL3342" (id 2) (at 247.65 60.96 0)
       (effects (font (size 1.27 1.27)) hide)
     )
@@
     )
     (path "/00000000-0000-0000-0000-0000609974e9/00000000-0000-0000-0000-00006099c285"
-      (reference "D201") (unit 1) (value "D_Zener") (footprint "Diode_SMD:D_0805_2012Metric_Pad1.15x1.40mm_HandSolder")
+      (reference "D201") (unit 1) (value "BZX284-C5V1") (footprint "Diode_SMD:D_SOD-110")
     )
     (path "/00000000-0000-0000-0000-000060a9ac30/00000000-0000-0000-0000-000060b67313"
@@
     )
     (path "/00000000-0000-0000-0000-0000609974e9/00000000-0000-0000-0000-000060998f82"
-      (reference "Q201") (unit 1) (value "Q_PMOS_GSD") (footprint "Package_TO_SOT_SMD:TSOT-23")
+      (reference "Q201") (unit 1) (value "SI4435DY_GSD") (footprint "Package_SO:SOIC-8_3.9x4.9mm_P1.27mm")
     )
     (path "/00000000-0000-0000-0000-000060968a02"
@@
       (reference "R202") (unit 1) (value "1M") (footprint "Resistor_SMD:R_0603_1608Metric_Pad0.98x0.95mm_HandSolder")
     )
+    (path "/00000000-0000-0000-0000-0000609974e9/a03d0f3d-c3fe-4e03-bb94-bcc91c33fae5"
+      (reference "R204") (unit 1) (value "100R") (footprint "Resistor_SMD:R_0603_1608Metric_Pad0.98x0.95mm_HandSolder")
+    )
     (path "/00000000-0000-0000-0000-0000609974e9/00000000-0000-0000-0000-0000615f098e"
       (reference "R210") (unit 1) (value "10") (footprint "Resistor_SMD:R_1206_3216Metric_Pad1.30x1.75mm_HandSolder")
@@
     )
     (path "/00000000-0000-0000-0000-00006095333e"
-      (reference "SW1") (unit 1) (value "SW_Push") (footprint "Button_Switch_SMD:SW_Push_1P1T_NO_6x6mm_H9.5mm")
+      (reference "SW1") (unit 1) (value "SW_Push") (footprint "Button_Switch_THT:SW_PUSH_6mm_H5mm")
     )
     (path "/00000000-0000-0000-0000-000060953687"
-      (reference "SW2") (unit 1) (value "SW_Push") (footprint "Button_Switch_SMD:SW_Push_1P1T_NO_6x6mm_H9.5mm")
+      (reference "SW2") (unit 1) (value "SW_Push") (footprint "Button_Switch_THT:SW_PUSH_6mm_H5mm")
     )
     (path "/00000000-0000-0000-0000-0000609d2703"
-      (reference "SW3") (unit 1) (value "SW_Push") (footprint "Button_Switch_SMD:SW_Push_1P1T_NO_6x6mm_H9.5mm")
+      (reference "SW3") (unit 1) (value "SW_Push") (footprint "Button_Switch_THT:SW_PUSH_6mm_H5mm")
     )
     (path "/00000000-0000-0000-0000-000061b18aaf"
-      (reference "SW4") (unit 1) (value "SW_Push") (footprint "Button_Switch_SMD:SW_Push_1P1T_NO_6x6mm_H9.5mm")
+      (reference "SW4") (unit 1) (value "SW_Push") (footprint "Button_Switch_SMD:SW_SPST_TL3342")
     )
     (path "/00000000-0000-0000-0000-00006063995a"

Commit message: Updated power section. Updated all possible footprints to be "hand solder" version. Updated Symbol lib.
Parts:
- C100, C101, C102, C110: footprint Capacitor_SMD:C_0603_1608Metric -> Capacitor_SMD:C_0603_1608Metric_Pad1.08x0.95mm_HandSolder

Commit message: ... Forgot to connect the data line to esp32... It's done now.
Connections:
- net WS2812B-DATA: now reaches U1.31 (IO19)
- no-connect marks 20 -> 19
Changed lines of the file:
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@@
   (no_connect (at 87.63 83.82))
   (no_connect (at 87.63 91.44))
-  (no_connect (at 118.11 83.82))
   (no_connect (at 87.63 93.98))
   (no_connect (at 118.11 88.9))
@@
     (stroke (width 0) (type default) (color 0 0 0 0))
   )
+  (wire (pts (xy 118.11 83.82) (xy 124.46 83.82))
+    (stroke (width 0) (type default) (color 0 0 0 0))
+  )
   (wire (pts (xy 152.4 152.4) (xy 152.4 149.86))
     (stroke (width 0) (type default) (color 0 0 0 0))
@@
     )
   )
+  (global_label "WS2812B-DATA" (shape input) (at 124.46 83.82 0) (fields_autoplaced)
+    (effects (font (size 1.27 1.27)) (justify left))
+    (property "Intersheet References" "${INTERSHEET_REFS}" (id 0) (at 141.5404 83.7406 0)
+      (effects (font (size 1.27 1.27)) (justify left) hide)
+    )
+  )

Commit message: Fixed known errors. * Reset curcuit, know is pull high with button tieing it low * OP-amp now uses correct, larger, footprint.
Parts:
- added R13: 10, Resistor_SMD:R_0603_1608Metric_Pad0.98x0.95mm_HandSolder, symbol Device:R
- R101, R103: value 10k -> 10
Connections:
- net GND: now also R13.2
- net RESET: now also R111.2
- net at SW4.2: now also R13.1; no longer R111.2
Other:
- moved on the sheet: R111
Changed lines of the file:
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@@
     (stroke (width 0) (type default) (color 0 0 0 0))
   )
-  (wire (pts (xy 257.81 58.42) (xy 257.81 55.88))
+  (wire (pts (xy 237.49 58.42) (xy 237.49 55.88))
     (stroke (width 0) (type default) (color 0 0 0 0))
   )
@@
       (effects (font (size 1.27 1.27)) (justify left))
     )
-    (property "Value" "10k" (id 1) (at 203.708 27.2666 0)
+    (property "Value" "10" (id 1) (at 203.708 27.2666 0)
       (effects (font (size 1.27 1.27)) (justify left))
     )
@@
       (effects (font (size 1.27 1.27)) (justify left))
     )
-    (property "Value" "10k" (id 1) (at 203.708 47.5866 0)
+    (property "Value" "10" (id 1) (at 203.708 47.5866 0)
       (effects (font (size 1.27 1.27)) (justify left))
     )
@@
     (pin "2")
   )
-  (symbol (lib_id "Device:R") (at 257.81 62.23 0) (unit 1)
-    (in_bom yes) (on_board yes)
-    (property "Reference" "R111" (id 0) (at 259.588 61.0616 0)
-      (effects (font (size 1.27 1.27)) (justify left))
-    )
-    (property "Value" "10k" (id 1) (at 259.588 63.373 0)
-      (effects (font (size 1.27 1.27)) (justify left))
-    )
-    (property "Footprint" "Resistor_SMD:R_0603_1608Metric_Pad0.98x0.95mm_HandSolder" (id 2) (at 256.032 62.23 90)
-      (effects (font (size 1.27 1.27)) hide)
-    )
-    (property "Datasheet" "~" (id 3) (at 257.81 62.23 0)
-      (effects (font (size 1.27 1.27)) hide)
-    )
-    (pin "1")
-    (pin "2")
-  )
-  (symbol (lib_id "power:+3V3") (at 257.81 55.88 0) (unit 1)
-    (in_bom yes) (on_board yes)
-    (property "Reference" "#PWR0208" (id 0) (at 257.81 59.69 0)
-      (effects (font (size 1.27 1.27)) hide)
-    )
-    (property "Value" "+3V3" (id 1) (at 258.191 51.4858 0))
-    (property "Footprint" "" (id 2) (at 257.81 55.88 0)
-      (effects (font (size 1.27 1.27)) hide)
-    )
-    (property "Datasheet" "" (id 3) (at 257.81 55.88 0)
+  (symbol (lib_id "Device:R") (at 237.49 62.23 0) (unit 1)
+    (in_bom yes) (on_board yes)
+    (property "Reference" "R111" (id 0) (at 239.268 61.0616 0)
+      (effects (font (size 1.27 1.27)) (justify left))
+    )
+    (property "Value" "10k" (id 1) (at 239.268 63.373 0)
+      (effects (font (size 1.27 1.27)) (justify left))
+    )
+    (property "Footprint" "Resistor_SMD:R_0603_1608Metric_Pad0.98x0.95mm_HandSolder" (id 2) (at 235.712 62.23 90)
+      (effects (font (size 1.27 1.27)) hide)
+    )
+    (property "Datasheet" "~" (id 3) (at 237.49 62.23 0)
+      (effects (font (size 1.27 1.27)) hide)
+    )
+    (pin "1")
+    (pin "2")
+  )
+  (symbol (lib_id "power:+3V3") (at 237.49 55.88 0) (unit 1)
+    (in_bom yes) (on_board yes)
+    (property "Reference" "#PWR0208" (id 0) (at 237.49 59.69 0)
+      (effects (font (size 1.27 1.27)) hide)
+    )
+    (property "Value" "+3V3" (id 1) (at 237.871 51.4858 0))
+    (property "Footprint" "" (id 2) (at 237.49 55.88 0)
+      (effects (font (size 1.27 1.27)) hide)
+    )
+    (property "Datasheet" "" (id 3) (at 237.49 55.88 0)
       (effects (font (size 1.27 1.27)) hide)
     )
@@
     (pin "1")
     (pin "2")
+  )
+  (symbol (lib_id "Device:R") (at 257.81 69.85 0) (unit 1)
+    (in_bom yes) (on_board yes)
+    (property "Reference" "R13" (id 0) (at 259.588 68.6816 0)
+      (effects (font (size 1.27 1.27)) (justify left))
+    )
+    (property "Value" "10" (id 1) (at 259.588 70.993 0)
+      (effects (font (size 1.27 1.27)) (justify left))
+    )
+    (property "Footprint" "Resistor_SMD:R_0603_1608Metric_Pad0.98x0.95mm_HandSolder" (id 2) (at 256.032 69.85 90)
+      (effects (font (size 1.27 1.27)) hide)
+    )
+    (property "Datasheet" "~" (id 3) (at 257.81 69.85 0)
+      (effects (font (size 1.27 1.27)) hide)
+    )
+    (pin "1")
+    (pin "2")
+  )
+  (symbol (lib_id "power:GND") (at 257.81 73.66 0) (unit 1)
+    (in_bom yes) (on_board yes)
+    (property "Reference" "#PWR0118" (id 0) (at 257.81 80.01 0)
+      (effects (font (size 1.27 1.27)) hide)
+    )
+    (property "Value" "GND" (id 1) (at 257.937 78.0542 0))
+    (property "Footprint" "" (id 2) (at 257.81 73.66 0)
+      (effects (font (size 1.27 1.27)) hide)
+    )
+    (property "Datasheet" "" (id 3) (at 257.81 73.66 0)
+      (effects (font (size 1.27 1.27)) hide)
+    )
+    (pin "1")
   )
   (sheet (at 24.13 157.48) (size 44.45 10.16) (fields_autoplaced)
@@
       (reference "#PWR0117") (unit 1) (value "GND") (footprint "")
     )
+    (path "/efa4fa83-e154-4feb-8823-0144c4836d67"
+      (reference "#PWR0118") (unit 1) (value "GND") (footprint "")
+    )
     (path "/00000000-0000-0000-0000-0000609974e9/00000000-0000-0000-0000-00006141906a"
       (reference "#PWR0119") (unit 1) (value "VCC") (footprint "")
@@
       (reference "R12") (unit 1) (value "100k") (footprint "Resistor_SMD:R_0603_1608Metric_Pad0.98x0.95mm_HandSolder")
     )
+    (path "/4aa6bf01-b5e0-4b67-b167-e7cec0b318d5"
+      (reference "R13") (unit 1) (value "10") (footprint "Resistor_SMD:R_0603_1608Metric_Pad0.98x0.95mm_HandSolder")
+    )
     (path "/00000000-0000-0000-0000-00006095d6fb"
-      (reference "R101") (unit 1) (value "10k") (footprint "Resistor_SMD:R_0603_1608Metric_Pad0.98x0.95mm_HandSolder")
+      (reference "R101") (unit 1) (value "10") (footprint "Resistor_SMD:R_0603_1608Metric_Pad0.98x0.95mm_HandSolder")
     )
     (path "/00000000-0000-0000-0000-00006095679c"
@@
     )
     (path "/00000000-0000-0000-0000-00006095d93c"
-      (reference "R103") (unit 1) (value "10k") (footprint "Resistor_SMD:R_0603_1608Metric_Pad0.98x0.95mm_HandSolder")
+      (reference "R103") (unit 1) (value "10") (footprint "Resistor_SMD:R_0603_1608Metric_Pad0.98x0.95mm_HandSolder")
     )
     (path "/00000000-0000-0000-0000-000060648800"
@@
     )
     (path "/00000000-0000-0000-0000-00006099554c/631167f5-11a2-46cd-80e9-ce323cd1eec7"
-      (reference "U2") (unit 1) (value "MCP6001x-LT") (footprint "Package_TO_SOT_SMD:SOT-353_SC-70-5")
+      (reference "U2") (unit 1) (value "MCP6001x-LT") (footprint "Package_TO_SOT_SMD:SOT-23-5")
     )
     (path "/00000000-0000-0000-0000-0000609974e9/00000000-0000-0000-0000-000061aeb8b2"
